Commit message: finish section 8

File: src/cpp_bumperbot/urdf/bumperbot.gazebo.xacro (robot description, xacro)
@@ -12,11 +12,4 @@
 		<actuator name="wheel_left_motor" role="actuator_left"/>
 		<joint name="wheel_left_joint" role="joint_left">
-			<mechanical_reduction>1.0</mechanical_reduction>
-		</joint>
-	</transmission>
-	<transmission name="can_transmission">
-		<plugin>transmission_interface/SimpleTransmission</plugin>
-		<actuator name="can_motor" role="actuator_can"/>
-		<joint name="can_joint" role="joint_can">
 			<mechanical_reduction>1.0</mechanical_reduction>
 		</joint>

File: src/cpp_bumperbot/urdf/bumperbot.urdf.xacro (robot description, xacro)
@@ -157,9 +157,8 @@
 		</collision>
 	</link>
-	<joint name="can_joint" type="continuous">
+	<joint name="can_joint" type="fixed">
 		<parent link="base_link" />
 		<child link="can_link" />
 		<origin rpy="0 0 0" xyz="0 0 0.078" />
-		<axis xyz="1 0 0" />
 	</joint>
 </robot>

File: src/cpp_bumperbot/urdf/bumperbot_ros2_control.xacro (robot description, xacro)
@@ -21,12 +21,4 @@
 			<state_interface name="velocity" />
 		</joint>
-		<joint name="can_joint">
-			<command_interface name="velocity">
-				<param name="min">-1</param>
-				<param name="max">1</param>
-			</command_interface>
-			<state_interface name="position" />
-			<state_interface name="velocity" />
-		</joint>
 	</ros2_control>
 </robot>
