Commit message: new modified

File: src/robot_description/urdf/robot.urdf.xacro (robot description, xacro)
@@ -1,5 +1,11 @@
 <?xml version="1.0" ?>
 <robot xmlns:xacro="http://www.ros.org/wiki/xacro" name="robot">
+	<!-- load parameters from launch file -->
+	<xacro:arg name="is_simulate" default="true" />
+	<!-- load from other xacro files -->
 	<xacro:include filename="robot_core.xacro" />
+	<xacro:if value="$(arg is_simulate)">
+		<xacro:include filename="gazebo.xacro" />
+	</xacro:if>
 	<xacro:include filename="ros2_control.xacro" />
 </robot>

File: src/robot_description/urdf/robot_core.xacro (robot description, xacro)
@@ -3,41 +3,160 @@
 	<link name="base_footprint" />
 	<link name="base_link" >
+		<inertial>
+			<origin xyz="0 0 0.04" rpy="0.0 0.25 0.3" />
+			<mass value="8.2573504e-01" />
+			<inertia ixx="2.2124416e-02" ixy="-1.2294101e-04" ixz="3.4938785e-04"
+					 iyy="2.1193702e-02" iyz="-5.0120904e-05"
+					 izz="2.0064271e-02" />
+		</inertial>
 		<visual>
-			<origin rpy="0 0 0" xyz="0 0 1"/>
+			<origin rpy="0 0 0" xyz="0 0 0"/>
 			<geometry>
-				<sphere radius="0.01"/>
+				<mesh filename="package://cpp_bumperbot/meshes/base_link.STL" />
 			</geometry>
 		</visual>
+		<collision>
+			<origin rpy="0 0 0" xyz="0 0 0"/>
+			<geometry>
+				<mesh filename="package://cpp_bumperbot/meshes/base_link.STL" />
+			</geometry>
+		</collision>
 	</link>
 	<joint name="base_joint" type="fixed">
 		<parent link="base_footprint" />
 		<child link="base_link" />
-		<origin rpy="0 0 0" xyz="0 0 0.05" />
+		<origin rpy="0 0 0" xyz="0 0 0.033" />
 	</joint>
-	<link name="wheel_left_link" >
+	<link name="wheel_right_link">
+		<inertial>
+			<origin xyz="0 -0.014 0" rpy="0 0 0" />
+			<mass value="0.0530086090966721" />
+			<inertia ixx="1.88176298336665E-05" ixy="-4.8444933029987E-10" ixz="1.88163708851143E-08"
+					 iyy="3.11510738647764E-05" iyz="-6.93560663069607E-11"
+					 izz="1.8801969558182E-05" />
+		</inertial>
 		<visual>
-			<origin rpy="0 0 0" xyz="-0.05 0 0"/>
+			<origin rpy="1.57 0 0" xyz="0 0 0"/>
+			<geometry>
+				<mesh filename="package://cpp_bumperbot/meshes/wheel_right_link.STL" />
+			</geometry>
+		</visual>
+		<collision>
+			<origin rpy="1.57 0 0" xyz="0 -0.015 0"/>
+			<geometry>
+				<sphere radius="0.033"/>
+			</geometry>
+		</collision>
+	</link>
+	<joint name="wheel_right_joint" type="continuous">
+		<parent link="base_link" />
+		<child link="wheel_right_link" />
+		<origin rpy="0 0 0" xyz="0 -0.07 0" />
+		<axis xyz="0 1 0" />
+	</joint>
+	<link name="wheel_left_link">
+		<inertial>
+			<origin xyz="0 0.014 0" rpy="0 0 0" />
+			<mass value="0.0530086043217644" />
+			<inertia ixx="1.8792911368909E-05"  ixy="3.31256392204584E-10" ixz="-1.14082001662767E-08"
+					 iyy="3.11510738759073E-05" iyz="-3.60499245082192E-10"
+					 izz="1.88266886146847E-05" />
+		</inertial>
+		<visual>
+			<origin rpy="-1.57 0 0" xyz="0 0 0"/>
+			<geometry>
+				<mesh filename="package://cpp_bumperbot/meshes/wheel_left_link.STL" />
+			</geometry>
+		</visual>
+		<collision>
+			<origin rpy="1.57 0 0" xyz="0 0.015 0"/>
+			<geometry>
+				<sphere radius="0.033"/>
+			</geometry>
+		</collision>
+	</link>
+	<joint name="wheel_left_joint" type="continuous">
+		<parent link="base_link" />
+		<child link="wheel_left_link" />
+		<origin rpy="0 0 0" xyz="0 0.07 0" />
+		<axis xyz="0 1 0" />
+	</joint>
+	<link name="caster_front_link">
+		<inertial>
+			<origin xyz="3.89968128948481E-07 2.40073004698083E-07 0.00219173397061506" rpy="0 0 0" />
+			<mass value="1.44379265037903E-06" />
+			<inertia ixx="7.23075276010246E-11" ixy="-6.10956883467859E-16" ixz="2.22849693525031E-15"
+					 iyy="3.8713793085917E-11"  iyz="2.93909858781952E-15"
+					 izz="1.00967486676306E-10" />
+		</inertial>
+		<visual>
+			<origin rpy="0 0 0" xyz="0 0 0"/>
+			<geometry>
+				<mesh filename="package://cpp_bumperbot/meshes/caster_front_link.STL" />
+			</geometry>
+		</visual>
+		<collision>
+			<origin rpy="0 0 0" xyz="0 0 0"/>
 			<geometry>
 				<sphere radius="0.005"/>
 			</geometry>
+		</collision>
+	</link>
+	<joint name="caster_front_joint" type="fixed">
+		<parent link="base_link" />
+		<child link="caster_front_link" />
+		<origin rpy="0 0 0" xyz="0.04755 0 -0.0275" />
+	</joint>
+	<link name="caster_rear_link">
+		<inertial>
+			<origin xyz="3.8996812895542E-07 2.40073004698083E-07 0.00219173397061509" rpy="0 0 0" />
+			<mass value="1.44379265037902E-06" />
+			<inertia ixx="7.23075276010246E-11" ixy="-6.10956872363424E-16" ixz="2.22849693527207E-15"
+					 iyy="3.87137930859167E-11" iyz="2.939098587861E-15"
+					 izz="1.00967486676306E-10" />
+		</inertial>
+		<visual>
+			<origin rpy="0 0 0" xyz="0 0 0"/>
+			<geometry>
+				<mesh filename="package://cpp_bumperbot/meshes/caster_rear_link.STL" />
+			</geometry>
 		</visual>
-	</link>
-	<link name="wheel_right_link" >
-		<visual>
-			<origin rpy="0 0 0" xyz="0.05 0 0"/>
+		<collision>
+			<origin rpy="0 0 0" xyz="0 0 0"/>
 			<geometry>
 				<sphere radius="0.005"/>
 			</geometry>
+		</collision>
+	</link>
+	<joint name="caster_rear_joint" type="fixed">
+		<parent link="base_link" />
+		<child link="caster_rear_link" />
+		<origin rpy="0 0 0" xyz="-0.047 0 -0.027" />
+	</joint>
+	<link name="can_link">
+		<inertial>
+			<origin xyz="3.8996812895542E-07 2.40073004698083E-07 0.00219173397061509" rpy="0 0 0" />
+			<mass value="1.44379265037902E-06" />
+			<inertia ixx="7.23075276010246E-11" ixy="-6.10956872363424E-16" ixz="2.22849693527207E-15"
+					 iyy="3.87137930859167E-11" iyz="2.939098587861E-15"
+					 izz="1.00967486676306E-10" />
+		</inertial>
+		<visual>
+			<origin rpy="1.57 0 0" xyz="-0.032 0.032 0"/>
+			<geometry>
+				<mesh filename="package://cpp_bumperbot/meshes/can_link.STL" />
+			</geometry>
 		</visual>
+		<collision>
+			<origin rpy="1.57 0 0" xyz="-0.032 0.032 0"/>
+			<geometry>
+				<sphere radius="0.01"/>
+			</geometry>
+		</collision>
 	</link>
-	<joint name="wheel_left_joint" type="fixed">
+	<joint name="can_joint" type="fixed">
 		<parent link="base_link" />
-		<child link="wheel_left_link" />
-		<origin rpy="0 0 0" xyz="-0.05 0 0" />
-	</joint>
-	<joint name="wheel_right_joint" type="fixed">
-		<parent link="base_link" />
-		<child link="wheel_right_link" />
-		<origin rpy="0 0 0" xyz="0.05 0 0" />
+		<child link="can_link" />
+		<origin rpy="0 0 0" xyz="0 0 0.078" />
 	</joint>
 </robot>

File: src/robot_description/urdf/ros2_control.xacro (robot description, xacro)
@@ -2,8 +2,16 @@
 <robot xmlns:xacro="http://www.ros.org/wiki/xacro">
 	<ros2_control name="RobotSystem" type="system">
-		<!-- load interfaces -->
-		<hardware>
-			<plugin>robot_firmware/WheelInterface</plugin>
-		</hardware>
+		<!-- ros2_control in gazebo env -->
+		<xacro:if value="$(arg is_simulate)">
+			<hardware>
+				<plugin>gazebo_ros2_control/GazeboSystem</plugin>
+			</hardware>
+		</xacro:if>
+		<!-- load interfaces for real robot -->
+		<xacro:unless value="$(arg is_simulate)">
+			<hardware>
+				<plugin>robot_firmware/WheelInterface</plugin>
+			</hardware>
+		</xacro:unless>
 		<!-- define joints and interfaces -->
 		<joint name="wheel_left_joint">

Commit message: add mpu6050 and params to launch files

File: src/robot_description/urdf/robot.urdf.xacro (robot description, xacro)
@@ -2,8 +2,8 @@
 <robot xmlns:xacro="http://www.ros.org/wiki/xacro" name="robot">
 	<!-- load parameters from launch file -->
-	<xacro:arg name="is_simulate" default="false" />
+	<xacro:arg name="is_simulate" default="no" />
 	<!-- load from other xacro files -->
 	<xacro:include filename="robot_core.xacro" />
-	<xacro:if value="$(arg is_simulate)">
+	<xacro:if value="${is_simulate == yes}">
 		<xacro:include filename="gazebo.xacro" />
 	</xacro:if>

File: src/robot_description/urdf/robot_core.xacro (robot description, xacro)
@@ -134,26 +134,26 @@
 		<origin rpy="0 0 0" xyz="-0.047 0 -0.027" />
 	</joint>
-	<!-- <link name="imu_link">
+	<link name="imu_link">
 		<inertial>
-		<origin xyz="-0.00552433659106688 0.000168210391520346 0.000514000497342681" rpy="0 0 0" />
-		<mass value="0.000528415362211671" />
-		<inertia ixx="1.46176048428261E-08" ixy="1.40015117949421E-10" ixz="-1.99633872937403E-12"
-				iyy="8.59662482954888E-09" iyz="7.52375112767959E-12"
-				izz="2.30279421279312E-08" />
+			<origin xyz="-0.00552433659106688 0.000168210391520346 0.000514000497342681" rpy="0 0 0" />
+			<mass value="0.000528415362211671" />
+			<inertia ixx="1.46176048428261E-08" ixy="1.40015117949421E-10" ixz="-1.99633872937403E-12"
+					iyy="8.59662482954888E-09" iyz="7.52375112767959E-12"
+					izz="2.30279421279312E-08" />
 		</inertial>
 		<visual>
-		<origin xyz="0 0 0" rpy="0 0 0" />
-		<geometry>
-			<mesh filename="package://robot_description/meshes/imu_link.STL" />
-		</geometry>
-		<material name="">
-			<color rgba="0.792156862745098 0.819607843137255 0.933333333333333 1" />
-		</material>
+			<origin xyz="0 0 0" rpy="0 0 0" />
+			<geometry>
+				<mesh filename="package://robot_description/meshes/imu_link.STL" />
+			</geometry>
+			<material name="">
+				<color rgba="0.792156862745098 0.819607843137255 0.933333333333333 1" />
+			</material>
 		</visual>
 		<collision>
-		<origin xyz="0 0 0" rpy="0 0 0" />
-		<geometry>
-			<mesh filename="package://robot_description/meshes/imu_link.STL" />
-		</geometry>
+			<origin xyz="0 0 0" rpy="0 0 0" />
+			<geometry>
+				<mesh filename="package://robot_description/meshes/imu_link.STL" />
+			</geometry>
 		</collision>
 	</link>
@@ -163,5 +163,5 @@
 		<child link="imu_link" />
 		<axis xyz="0 0 0" />
-	</joint> -->
+	</joint>
 	<!-- LIDAR -->
 	<link name="lidar_link">

File: src/robot_description/urdf/ros2_control.xacro (robot description, xacro)
@@ -1,7 +1,7 @@
 <?xml version="1.0" ?>
 <robot xmlns:xacro="http://www.ros.org/wiki/xacro">
-	<ros2_control name="RobotSystem" type="system">
+	<ros2_control name="MotionPart" type="system">
 		<!-- ros2_control interfaces in gazebo env -->
-		<xacro:if value="$(arg is_simulate)">
+		<xacro:if value="${is_simulate == yes}">
 			<hardware>
 				<plugin>gazebo_ros2_control/GazeboSystem</plugin>
@@ -9,5 +9,5 @@
 		</xacro:if>
 		<!-- load interfaces for real robot -->
-		<xacro:unless value="$(arg is_simulate)">
+		<xacro:unless value="${is_simulate == yes}">
 			<hardware>
 				<plugin>robot_firmware/WheelInterface</plugin>
@@ -32,3 +32,24 @@
 		</joint>
 	</ros2_control>
+	<xacro:unless value="${is_simulate == yes}">
+		<ros2_control name="SensorPart" type="sensor">
+			<hardware>
+				<plugin>robot_firmware/MPU6050Interface</plugin>
+				<param name="sensor_name">mpu6050</param>
+				<param name='frame_id'>imu_link</param>
+			</hardware>
+			<sensor name='mpu6050'>
+				<state_interface name='orientation.x'/>
+				<state_interface name='orientation.y'/>
+				<state_interface name='orientation.z'/>
+				<state_interface name='orientation.w'/>
+				<state_interface name='angular_velocity.x'/>
+				<state_interface name='angular_velocity.y'/>
+				<state_interface name='angular_velocity.z'/>
+				<state_interface name='linear_acceleration.x'/>
+				<state_interface name='linear_acceleration.y'/>
+				<state_interface name='linear_acceleration.z'/>
+			</sensor>
+		</ros2_control>
+	</xacro:unless>
 </robot>

Commit message: Fix TF done. Scanning map and loading map

File: src/robot_description/urdf/robot.urdf.xacro (robot description, xacro)
@@ -2,8 +2,8 @@
 <robot xmlns:xacro="http://www.ros.org/wiki/xacro" name="robot">
 	<!-- load parameters from launch file -->
-	<xacro:arg name="is_simulate" default="no" />
+	<xacro:arg name="is_simulate" default="false" />
 	<!-- load from other xacro files -->
-	<xacro:include filename="robot_core.xacro" />
-	<xacro:if value="${is_simulate == yes}">
+	<xacro:include filename="test_core.xacro" />
+	<xacro:if value="$(arg is_simulate)">
 		<xacro:include filename="gazebo.xacro" />
 	</xacro:if>

File: src/robot_description/urdf/robot_core.xacro (robot description, xacro)
@@ -162,5 +162,5 @@
 		<parent link="base_link" />
 		<child link="imu_link" />
-		<axis xyz="0 0 0" />
+		<!-- <axis xyz="0 0 0" /> -->
 	</joint>
 	<!-- LIDAR -->
@@ -186,5 +186,5 @@
 		<child link="lidar_link"/>
 		<origin xyz="0.0 0.0 0.08" rpy="0 0 0"/>
-		<axis xyz="0 0 1"/>
+		<!-- <axis xyz="0 0 1"/> -->
 	</joint>
 </robot>

File: src/robot_description/urdf/ros2_control.xacro (robot description, xacro)
@@ -3,5 +3,5 @@
 	<ros2_control name="MotionPart" type="system">
 		<!-- ros2_control interfaces in gazebo env -->
-		<xacro:if value="${is_simulate == yes}">
+		<xacro:if value="$(arg is_simulate)">
 			<hardware>
 				<plugin>gazebo_ros2_control/GazeboSystem</plugin>
@@ -9,5 +9,5 @@
 		</xacro:if>
 		<!-- load interfaces for real robot -->
-		<xacro:unless value="${is_simulate == yes}">
+		<xacro:unless value="$(arg is_simulate)">
 			<hardware>
 				<plugin>robot_firmware/WheelInterface</plugin>
@@ -32,5 +32,5 @@
 		</joint>
 	</ros2_control>
-	<xacro:unless value="${is_simulate == yes}">
+	<xacro:unless value="$(arg is_simulate)">
 		<ros2_control name="SensorPart" type="sensor">
 			<hardware>
