Commit message: add new ROS2_control controller and interface to control broom

File: src/robot_description/urdf/ros2_control.xacro (robot description, xacro)
@@ -1,4 +1,5 @@
 <?xml version="1.0" ?>
 <robot xmlns:xacro="http://www.ros.org/wiki/xacro">
+<xacro:if value="$(arg is_simulate)">
 	<ros2_control name="MotionPart" type="system">
 		<!-- ros2_control interfaces in gazebo env -->
@@ -32,5 +33,16 @@
 		</joint>
 	</ros2_control>
-	<xacro:unless value="$(arg is_simulate)">
+</xacro:if>
+	<ros2_control name="CleanPart" type="system">
+		<hardware>
+			<plugin>robot_firmware/MopInterface</plugin>
+		</hardware>
+		<joint name="mop_joint">
+			<command_interface name="velocity"/>
+			<state_interface name="position"/>
+		</joint>
+	</ros2_control>
+<xacro:if value="$(arg is_simulate)">
+	<!-- <xacro:unless value="$(arg is_simulate)">
 		<ros2_control name="SensorPart" type="sensor">
 			<hardware>
@@ -52,4 +64,5 @@
 			</sensor>
 		</ros2_control>
-	</xacro:unless>
+	</xacro:unless> -->
+</xacro:if>
 </robot>

File: src/robot_description/urdf/test_core.xacro (robot description, xacro)
@@ -244,4 +244,19 @@
     <origin xyz="0.045 0 0.0175" rpy="0 0 0"/>
   </joint>
+  <!-- Mop -->
+  <link name="mop_link">
+	<visual name="mop_visual">
+		<origin xyz="0.105 0 0.0175" rpy="0 0 0"/>
+		<geometry>
+			<cylinder length="0.06" radius="0.02"/>
+		</geometry>
+	</visual>
+  </link>
+  <joint name="mop_joint" type="continuous">
+    <parent link="base_link"/>
+	<child link="mop_link"/>
+	<origin xyz="0 0 0" rpy="0 0 0"/>
+	<axis xyz="0 0 1"/>
+  </joint>
   <!-- <gazebo reference="caster_wheel">
     <mu1 value="0.001"/>
