Commit message: rewrite gazebo with ros2_controller

File: src/robot_description/urdf/gazebo.xacro (robot description, xacro)
@@ -1,4 +1,4 @@
 <?xml version="1.0"?>
-<robot name="bumperbot" xmlns:xacro="http://ros.org/wiki/xacro">
+<robot xmlns:xacro="http://ros.org/wiki/xacro">
   <!-- Move this one to ros2 control -->
   <transmission name="wheel_right_transmission">
@@ -52,10 +52,11 @@
     <maxVel>1.0</maxVel>
   </gazebo>
-  <!-- ROS 2 Control -->
+  <!-- add plugin for ROS2 Control -->
   <gazebo>
     <plugin filename="libgazebo_ros2_control.so" name="gazebo_ros2_control">
       <robot_param>robot_description</robot_param>
-      <robot_param_node>robot_state_publisher</robot_param_node>
-      <parameters>$(find bumperbot_controller)/config/bumperbot_controllers.yaml</parameters>
+      <robot_param_node>robot_state_publisher_node</robot_param_node>
+      <parameters>$(find robot_controller)/config/robot_controllers.yaml</parameters>
+      <controller_manager_name>simulation_controller_manager</controller_manager_name>
     </plugin>
   </gazebo>

File: src/robot_description/urdf/robot_core.xacro (robot description, xacro)
@@ -13,5 +13,5 @@
 			<origin rpy="0 0 0" xyz="0 0 0"/>
 			<geometry>
-				<mesh filename="package://cpp_bumperbot/meshes/base_link.STL" />
+				<mesh filename="package://robot_description/meshes/base_link.STL" />
 			</geometry>
 		</visual>
@@ -19,5 +19,5 @@
 			<origin rpy="0 0 0" xyz="0 0 0"/>
 			<geometry>
-				<mesh filename="package://cpp_bumperbot/meshes/base_link.STL" />
+				<mesh filename="package://robot_description/meshes/base_link.STL" />
 			</geometry>
 		</collision>
@@ -39,5 +39,5 @@
 			<origin rpy="1.57 0 0" xyz="0 0 0"/>
 			<geometry>
-				<mesh filename="package://cpp_bumperbot/meshes/wheel_right_link.STL" />
+				<mesh filename="package://robot_description/meshes/wheel_right_link.STL" />
 			</geometry>
 		</visual>
@@ -66,5 +66,5 @@
 			<origin rpy="-1.57 0 0" xyz="0 0 0"/>
 			<geometry>
-				<mesh filename="package://cpp_bumperbot/meshes/wheel_left_link.STL" />
+				<mesh filename="package://robot_description/meshes/wheel_left_link.STL" />
 			</geometry>
 		</visual>
@@ -93,5 +93,5 @@
 			<origin rpy="0 0 0" xyz="0 0 0"/>
 			<geometry>
-				<mesh filename="package://cpp_bumperbot/meshes/caster_front_link.STL" />
+				<mesh filename="package://robot_description/meshes/caster_front_link.STL" />
 			</geometry>
 		</visual>
@@ -119,5 +119,5 @@
 			<origin rpy="0 0 0" xyz="0 0 0"/>
 			<geometry>
-				<mesh filename="package://cpp_bumperbot/meshes/caster_rear_link.STL" />
+				<mesh filename="package://robot_description/meshes/caster_rear_link.STL" />
 			</geometry>
 		</visual>
@@ -145,5 +145,5 @@
 			<origin rpy="1.57 0 0" xyz="-0.032 0.032 0"/>
 			<geometry>
-				<mesh filename="package://cpp_bumperbot/meshes/can_link.STL" />
+				<mesh filename="package://robot_description/meshes/can_link.STL" />
 			</geometry>
 		</visual>

File: src/robot_description/urdf/ros2_control.xacro (robot description, xacro)
@@ -2,16 +2,16 @@
 <robot xmlns:xacro="http://www.ros.org/wiki/xacro">
 	<ros2_control name="RobotSystem" type="system">
-		<!-- ros2_control in gazebo env -->
-		<xacro:if value="$(arg is_simulate)">
+		<!-- ros2_control interfaces in gazebo env -->
+		<!-- <xacro:if value="$(arg is_simulate)"> -->
 			<hardware>
 				<plugin>gazebo_ros2_control/GazeboSystem</plugin>
 			</hardware>
-		</xacro:if>
+		<!-- </xacro:if> -->
 		<!-- load interfaces for real robot -->
-		<xacro:unless value="$(arg is_simulate)">
-			<hardware>
+		<!-- <xacro:unless value="$(arg is_simulate)"> -->
+			<!-- <hardware>
 				<plugin>robot_firmware/WheelInterface</plugin>
-			</hardware>
-		</xacro:unless>
+			</hardware> -->
+		<!-- </xacro:unless> -->
 		<!-- define joints and interfaces -->
 		<joint name="wheel_left_joint">

Commit message: ros2_control + nav2 + gazebo first success

File: src/robot_description/urdf/gazebo.xacro (robot description, xacro)
@@ -52,5 +52,5 @@
     <maxVel>1.0</maxVel>
   </gazebo>
-  <!-- add plugin for ROS2 Control -->
+  <!-- Ros2 Controller manager in Gazebo -->
   <gazebo>
     <plugin filename="libgazebo_ros2_control.so" name="gazebo_ros2_control">
@@ -61,6 +61,12 @@
     </plugin>
   </gazebo>
+  <!-- ros2_control interfaces in gazebo env -->
+  <!-- <xacro:if value="$(arg is_simulate)"> -->
+    <!-- <hardware>
+      <plugin>gazebo_ros2_control/GazeboSystem</plugin>
+    </hardware> -->
+  <!-- </xacro:if> -->
   <!-- IMU -->
-  <gazebo reference="imu_link">
+  <!-- <gazebo reference="imu_link">
     <sensor name="imu" type="imu">
         <always_on>true</always_on>
@@ -110,4 +116,39 @@
         <plugin name="imu" filename="libgazebo_ros_imu_sensor.so"/>
     </sensor>
+  </gazebo> -->
+  <gazebo reference="lidar_link">
+    <sensor name="lidar" type="ray">
+      <pose>0 0 0 0 0 0</pose>
+      <always_on>true</always_on>
+      <visualize>false</visualize>
+      <update_rate>10</update_rate>
+      <ray>
+          <scan>
+              <horizontal>
+                  <samples>360</samples>
+                  <min_angle>-3.14</min_angle>
+                  <max_angle>3.14</max_angle>
+              </horizontal>
+          </scan>
+          <range>
+              <min>0.15</min>
+              <max>6.0</max>
+              <!-- <max>12.0</max> -->
+              <resolution>0.01500</resolution>
+	      </range>
+          <noise>
+              <type>gaussian</type>
+              <mean>0.0</mean>
+              <stddev>0.01</stddev>
+          </noise>
+      </ray>
+      <plugin name="lidar_controller" filename="libgazebo_ros_ray_sensor.so">
+          <ros>
+              <remapping>~/out:=scan</remapping>
+          </ros>
+          <output_type>sensor_msgs/LaserScan</output_type>
+          <frame_name>lidar_link</frame_name>
+      </plugin>
+    </sensor>
   </gazebo>
 </robot>

File: src/robot_description/urdf/robot_core.xacro (robot description, xacro)
@@ -134,29 +134,57 @@
 		<origin rpy="0 0 0" xyz="-0.047 0 -0.027" />
 	</joint>
-	<link name="can_link">
+	<!-- <link name="imu_link">
 		<inertial>
-			<origin xyz="3.8996812895542E-07 2.40073004698083E-07 0.00219173397061509" rpy="0 0 0" />
-			<mass value="1.44379265037902E-06" />
-			<inertia ixx="7.23075276010246E-11" ixy="-6.10956872363424E-16" ixz="2.22849693527207E-15"
-					 iyy="3.87137930859167E-11" iyz="2.939098587861E-15"
-					 izz="1.00967486676306E-10" />
+		<origin xyz="-0.00552433659106688 0.000168210391520346 0.000514000497342681" rpy="0 0 0" />
+		<mass value="0.000528415362211671" />
+		<inertia ixx="1.46176048428261E-08" ixy="1.40015117949421E-10" ixz="-1.99633872937403E-12"
+				iyy="8.59662482954888E-09" iyz="7.52375112767959E-12"
+				izz="2.30279421279312E-08" />
 		</inertial>
 		<visual>
-			<origin rpy="1.57 0 0" xyz="-0.032 0.032 0"/>
+		<origin xyz="0 0 0" rpy="0 0 0" />
+		<geometry>
+			<mesh filename="package://robot_description/meshes/imu_link.STL" />
+		</geometry>
+		<material name="">
+			<color rgba="0.792156862745098 0.819607843137255 0.933333333333333 1" />
+		</material>
+		</visual>
+		<collision>
+		<origin xyz="0 0 0" rpy="0 0 0" />
+		<geometry>
+			<mesh filename="package://robot_description/meshes/imu_link.STL" />
+		</geometry>
+		</collision>
+	</link>
+	<joint name="imu_joint" type="fixed">
+		<origin xyz="0 0 0.0698986241758014" rpy="0 0 0" />
+		<parent link="base_link" />
+		<child link="imu_link" />
+		<axis xyz="0 0 0" />
+	</joint> -->
+	<!-- LIDAR -->
+	<link name="lidar_link">
+		<visual>
+			<origin xyz="0 0 0" rpy="0 0 0"/>
 			<geometry>
-				<mesh filename="package://robot_description/meshes/can_link.STL" />
+				<mesh filename="package://robot_description/meshes/rplidar_top.dae"/>
 			</geometry>
 		</visual>
 		<collision>
-			<origin rpy="1.57 0 0" xyz="-0.032 0.032 0"/>
+			<origin xyz="0 0 0" rpy="0 0 0"/>
 			<geometry>
-				<sphere radius="0.01"/>
+				<cylinder radius="0.037" length="0.021"/>
 			</geometry>
 		</collision>
+		<!-- <xacro:cylinder_inertia mass="0.07" length="0.021" radius="0.037">
+			<origin xyz="0 0 0" rpy="0 0 0"/>
+		</xacro:cylinder_inertia> -->
 	</link>
-	<joint name="can_joint" type="fixed">
-		<parent link="base_link" />
-		<child link="can_link" />
-		<origin rpy="0 0 0" xyz="0 0 0.078" />
+	<joint name="lidar_joint" type="fixed">
+		<parent link="base_link"/>
+		<child link="lidar_link"/>
+		<origin xyz="0.0 0.0 0.08" rpy="0 0 0"/>
+		<axis xyz="0 0 1"/>
 	</joint>
 </robot>

Commit message: seperate sim and real launch

File: src/robot_description/urdf/gazebo.xacro (robot description, xacro)
@@ -60,6 +60,26 @@
     </plugin>
   </gazebo>
+  <!-- DIFF DRIVE -->
+  <gazebo>
+    <plugin name="gazebo_wheel_controller" filename="libgazebo_ros_diff_drive.so">
+      <!-- <commandTopic>gazebo_wheel_controller/cmd_vel_unstamped</commandTopic> -->
+      <!-- Wheel information -->
+      <left_joint>wheel_left_joint</left_joint>
+      <right_joint>wheel_right_joint</right_joint>
+      <wheel_separation>0.134</wheel_separation>
+      <wheel_diameter>0.067</wheel_diameter>
+      <!-- Limits (can be adjusted later on)-->
+      <max_wheel_torque>20</max_wheel_torque>
+      <max_wheel_acceleration>2</max_wheel_acceleration>
+      <!-- Output -->
+      <odometry_frame>odom</odometry_frame>
+      <robot_base_frame>base_footprint</robot_base_frame>
+      <publish_odom>true</publish_odom>
+      <publish_odom_tf>true</publish_odom_tf>
+      <publish_wheel_tf>true</publish_wheel_tf>
+    </plugin>
+  </gazebo>
   <!-- IMU -->
-  <!-- <gazebo reference="imu_link">
+  <gazebo reference="imu_link">
     <sensor name="imu" type="imu">
         <always_on>true</always_on>
@@ -107,7 +127,8 @@
           </linear_acceleration>
         </imu>
-        <plugin name="imu" filename="libgazebo_ros_imu_sensor.so"/>
+        <plugin name="gazebo_imu" filename="libgazebo_ros_imu_sensor.so"/>
     </sensor>
-  </gazebo> -->
+  </gazebo>
+  <!-- LIDAR -->
   <gazebo reference="lidar_link">
     <sensor name="lidar" type="ray">

File: src/robot_description/urdf/ros2_control.xacro (robot description, xacro)
@@ -1,5 +1,4 @@
 <?xml version="1.0" ?>
 <robot xmlns:xacro="http://www.ros.org/wiki/xacro">
-<xacro:if value="$(arg is_simulate)">
 	<ros2_control name="MotionPart" type="system">
 		<!-- ros2_control interfaces in gazebo env -->
@@ -33,6 +32,5 @@
 		</joint>
 	</ros2_control>
-</xacro:if>
-	<ros2_control name="CleanPart" type="system">
+	<!-- <ros2_control name="CleanPart" type="system">
 		<hardware>
 			<plugin>robot_firmware/MopInterface</plugin>
@@ -42,7 +40,6 @@
 			<state_interface name="position"/>
 		</joint>
-	</ros2_control>
-<xacro:if value="$(arg is_simulate)">
-	<!-- <xacro:unless value="$(arg is_simulate)">
+	</ros2_control> -->
+	<xacro:unless value="$(arg is_simulate)">
 		<ros2_control name="SensorPart" type="sensor">
 			<hardware>
@@ -64,5 +61,4 @@
 			</sensor>
 		</ros2_control>
-	</xacro:unless> -->
-</xacro:if>
+	</xacro:unless>
 </robot>

File: src/robot_description/urdf/test_core.xacro (robot description, xacro)
@@ -245,5 +245,5 @@
   </joint>
   <!-- Mop -->
-  <link name="mop_link">
+  <!-- <link name="mop_link">
 	<visual name="mop_visual">
 		<origin xyz="0.105 0 0.0175" rpy="0 0 0"/>
@@ -258,5 +258,5 @@
 	<origin xyz="0 0 0" rpy="0 0 0"/>
 	<axis xyz="0 0 1"/>
-  </joint>
+  </joint> -->
   <!-- <gazebo reference="caster_wheel">
     <mu1 value="0.001"/>
